File: PCB_V2/esp_v2.kicad_pcb (KiCad board)
At the start: 2 copper layers, 86 x 67.5 mm, 13 parts, among them J2 Conn_01x03_Socket, J3 Screw_Terminal_01x02, U1 ESP-32S

Commit message: testseted model on nocdemcu
Parts:
- added D1: LED, LED_THT:LED_D1.8mm_W3.3mm_H2.4mm, F.Cu at (100.0, 60.0)
- added R1: 330, Resistor_SMD:R_0815_2038Metric_Pad1.20x4.05mm_HandSolder, F.Cu at (100.0, 65.0)
- added SW1: SW_SPST, Button_Switch_SMD:SW_DIP_SPSTx01_Slide_6.7x4.1mm_W8.61mm_P2.54mm_LowProfile, F.Cu at (90.0, 65.0)
- moved J3 12.5 mm to (71.5, 65.0)
Connections:
- FTDI1 pad 2: VCC -> SW
- U1 pad 2: VCC -> SW
Routing:
- net VCC: track 151.3 -> 75.1 mm
- net SW: track 0.00 -> 70.3 mm
- net GND: track 139.5 -> 150.5 mm
- net Net-(D1-A): track 0.00 -> 5.03 mm
Other:
- board size 86 x 67.5 mm -> 86 x 74.8 mm
